Commit message: Node vision for Ergo et Torso

File: install/share/poppy_torso_description/urdf/poppy_torso.urdf.xacro (robot description, xacro)
@@ -1,26 +1,686 @@
-<?xml version="1.0"?>
+<?xml version="1.0" encoding="utf-8"?>
 <robot xmlns:xacro="http://www.ros.org/wiki/xacro" name="poppy_torso">
   <!-- Properties -->
   <xacro:property name="namespace" value="poppy_torso" />
-<xacro:if value="$(arg fixed)">
-<link name="world"/>
-  <joint name="fixed" type="fixed">
-    <parent link="world"/>
-    <child link="base_link"/>
-  </joint>
-</xacro:if>
- <link name="base_link">
-    <visual>
-      <origin xyz="0 0 0" rpy="0 0 0" />
-      <geometry>
-        <mesh filename="package://poppy_torso_description/meshes/base_visual.STL" />
-      </geometry>
-    </visual>
-    <xacro:if value="${is_fixed == 'false'}">
-    <inertial>
-      <mass value="0.304441048219244" />
-      <inertia ixx="0.000444379589701896" iyy="0.00048561348802354" izz="0.000421911604661064" ixy="1.65486746667917E-08" ixz="-3.86276516415689E-09" iyz="2.15649474149961E-05" />
-    </inertial>
-    </xacro:if>
-  </link>
+  <xacro:arg name="fixed" default="true"/>
+  <xacro:property name="is_fixed" value="true"/>
+  <!-- Macro to add a camera. -->
+  <xacro:macro name="camera_macro"
+    params="namespace parent_link camera_suffix frame_rate
+      horizontal_fov image_width image_height image_format min_distance
+      max_distance noise_mean noise_stddev enable_visual *cylinder *origin">
+    <link name="${namespace}/camera_${camera_suffix}_link">
+      <!-- <collision> -->
+      <!--   <origin xyz="0 0 0" rpy="0 0 0" /> -->
+      <!--   <geometry> -->
+      <!--     <xacro:insert_block name="cylinder" /> -->
+      <!--   </geometry> -->
+      <!-- </collision> -->
+      <xacro:if value="${enable_visual}">
+        <visual>
+          <origin xyz="0 0 0" rpy="0 1.57079632679 0" />
+          <geometry>
+            <xacro:insert_block name="cylinder" />
+          </geometry>
+          <material name="red">
+		     <color rgba="1 0 0 1"/>
+	  </material>
+        </visual>
+      </xacro:if>
+      <inertial>
+        <mass value="1e-5" />
+        <origin xyz="0 0 0" rpy="0 0 0" />
+        <inertia ixx="1e-6" ixy="0" ixz="0" iyy="1e-6" iyz="0" izz="1e-6" />
+      </inertial>
+    </link>
+    <joint name="${namespace}/camera_${camera_suffix}_joint" type="fixed">
+      <xacro:insert_block name="origin" />
+      <parent link="${parent_link}" />
+      <child link="${namespace}/camera_${camera_suffix}_link" />
+    </joint>
+    <gazebo reference="${namespace}/camera_${camera_suffix}_link">
+      <sensor type="camera" name="${namespace}_camera_${camera_suffix}">
+        <update_rate>${frame_rate}</update_rate>
+        <camera name="head">
+          <horizontal_fov>${horizontal_fov}</horizontal_fov>
+          <image>
+            <width>${image_width}</width>
+            <height>${image_height}</height>
+            <format>${image_format}</format>
+          </image>
+          <clip>
+            <near>${min_distance}</near>
+            <far>${max_distance}</far>
+          </clip>
+          <noise>
+            <type>gaussian</type>
+            <!-- Noise is sampled independently per pixel on each frame.
+                 That pixel's noise value is added to each of its color
+                 channels, which at that point lie in the range [0,1]. -->
+            <mean>${noise_mean}</mean>
+            <stddev>${noise_stddev}</stddev>
+          </noise>
+        </camera>
+        <plugin name="${namespace}_camera_${camera_suffix}_controller" filename="libgazebo_ros_camera.so">
+          <robotNamespace>${namespace}</robotNamespace>
+          <alwaysOn>true</alwaysOn>
+          <updateRate>${frame_rate}</updateRate>
+          <cameraName>camera_${camera_suffix}</cameraName>
+          <imageTopicName>image_raw</imageTopicName>
+          <cameraInfoTopicName>camera_info</cameraInfoTopicName>
+          <frameName>camera_${camera_suffix}_link</frameName>
+          <hackBaseline>0.0</hackBaseline>
+	  <Cx>2.0500638605704751e+02</Cx>
+	  <Cy>1.5106876398089261e+02</Cy>
+	  <focalLength>632.193308</focalLength>
+          <distortionK1>1.4043219721770492e-01</distortionK1>
+          <distortionK2>-1.3210129724889583e-01</distortionK2>
+          <distortionK3>-3.6452869939025279e-01</distortionK3>
+          <distortionT1>-5.1782301614838704e-04</distortionT1>
+          <distortionT2>-5.2090817919999092e-03</distortionT2>
+        </plugin>
+      </sensor>
+    </gazebo>
+  </xacro:macro>
+<xacro:camera_macro
+    namespace="${namespace}"
+    parent_link="head"
+    camera_suffix="torso"
+    frame_rate="30.0"
+    horizontal_fov="1.12825740656329"
+    image_width="800"
+    image_height="600"
+    image_format="R8G8B8"
+    min_distance="0.02"
+    max_distance="400"
+    noise_mean="0.0"
+    noise_stddev="0.001"
+    enable_visual="true"
+    >
+    <!-- <box size="0.01 0.01 0.01" /> -->
+    <cylinder length="0.01" radius="0.007" />
+    <origin xyz="0 0.08 0.02" rpy="0 -1.57 -1.57"/>
+</xacro:camera_macro>
+	<gazebo>
+		<static>false</static>
+		<plugin name="gazebo_ros_control" filename="libgazebo_ros_control.so">
+			<robotNamespace>/poppy_torso</robotNamespace>
+			<robotSimType>gazebo_ros_control/DefaultRobotHWSim</robotSimType>
+			<legacyModeNS>true</legacyModeNS>
+		</plugin>
+	</gazebo>
+	<link name="world"/>
+	<link name="base">
+		<inertial>
+			<origin xyz="-9.74926801495556E-06 0.0245809270022031 -0.0126310576435619" rpy="0 0 0"></origin>
+			<mass value="0.304441048219244"></mass>
+			<inertia ixx="0.000444379589701896" ixy="1.65486746667917E-08" ixz="-3.86276516415689E-09" iyy="0.00048561348802354" iyz="2.15649474149961E-05" izz="0.000421911604661064"></inertia>
+		</inertial>
+		<visual>
+			<origin xyz="0 0 0" rpy="0 0 0"></origin>
+			<geometry>
+				<mesh filename="package://poppy_torso_description/meshes/base_visual.STL"></mesh>
+			</geometry>
+			<material name="">
+				<color rgba="0.9 0.9 0.9 1.0"></color>
+			</material>
+		</visual>
+		<collision>
+			<origin xyz="0 0 0" rpy="0 0 0"></origin>
+			<geometry>
+				<mesh filename="package://poppy_torso_description/meshes/base_respondable.STL"></mesh>
+			</geometry>
+		</collision>
+	</link>
+	<joint name="fixed" type="fixed">
+		<parent link="world"/>
+		<child link="base"/>
+	</joint>
+	<link name="spine">
+		<inertial>
+			<origin xyz="-2.40411891850495E-07 0.0288451667347867 -0.0100975118547382" rpy="0 0 0"></origin>
+			<mass value="0.0926815106655512"></mass>
+			<inertia ixx="3.84763910015325E-05" ixy="-1.20593001730888E-09" ixz="-2.38589260905183E-10" iyy="2.7320514654861E-05" iyz="1.47490149318973E-06" izz="3.26595211965373E-05"></inertia>
+		</inertial>
+		<visual>
+			<origin xyz="0 0 0" rpy="0 0 0"></origin>
+			<geometry>
+				<mesh filename="package://poppy_torso_description/meshes/spine_visual.STL"></mesh>
+			</geometry>
+			<material name="">
+				<color rgba="0.9 0.9 0.9 1.0"></color>
+			</material>
+		</visual>
+		<collision>
+			<origin xyz="0 0 0" rpy="0 0 0"></origin>
+			<geometry>
+				<mesh filename="package://poppy_torso_description/meshes/spine_respondable.STL"></mesh>
+			</geometry>
+		</collision>
+		<mass>0.09264</mass>
+	</link>
+	<joint name="abs_z" type="revolute">
+		<origin xyz="0 0 0.08965" rpy="1.5708 1.1258E-18 0.018388"></origin>
+		<parent link="base"></parent>
+		<child link="spine"></child>
+		<axis xyz="0 1 0"></axis>
+		<limit lower="-1.57079" upper="1.57079" effort="10" velocity="3.1415"></limit>
+	</joint>
+	<transmission name="abs_z_trans">
+		<type>transmission_interface/SimpleTransmission</type>
+		<joint name="abs_z">
+			<hardwareInterface>hardware_interface/PositionJointInterface</hardwareInterface>
+		</joint>
+		<actuator name="abs_z_motor">
+			<mechanicalReduction>1</mechanicalReduction>
+		</actuator>
+	</transmission>
+	<link name="bust_motors">
+		<inertial>
+			<origin xyz="3.50872416629779E-05 0.0105220286877652 -0.0174331453843439" rpy="0 0 0"></origin>
+			<mass value="0.158876054570625"></mass>
+			<inertia ixx="0.000100953683249293" ixy="-3.89105307189684E-07" ixz="9.71749941401585E-08" iyy="8.94288410563621E-05" iyz="-1.31738255727689E-06" izz="4.26225972692235E-05"></inertia>
+		</inertial>
+		<visual>
+			<origin xyz="0 0 0" rpy="0 0 0"></origin>
+			<geometry>
+				<mesh filename="package://poppy_torso_description/meshes/bust_motors_visual.STL"></mesh>
+			</geometry>
+			<material name="">
+				<color rgba="0.9 0.9 0.9 1.0"></color>
+			</material>
+		</visual>
+		<collision>
+			<origin xyz="0 0 0" rpy="0 0 0"></origin>
+			<geometry>
+				<mesh filename="package://poppy_torso_description/meshes/bust_motors_respondable.STL"></mesh>
+			</geometry>
+		</collision>
+		<mass>0.15889</mass>
+	</link>
+	<joint name="bust_y" type="revolute">
+		<origin xyz="0 0.07985 0.00279999999999998" rpy="0 0 0"></origin>
+		<parent link="spine"></parent>
+		<child link="bust_motors"></child>
+		<axis xyz="-1 0 0"></axis>
+		<limit lower="-1.0" upper="0.44" effort="10" velocity="3.1415"></limit>
+	</joint>
+	<transmission name="bust_y_trans">
+		<type>transmission_interface/SimpleTransmission</type>
+		<joint name="bust_y">
+			<hardwareInterface>hardware_interface/PositionJointInterface</hardwareInterface>
+		</joint>
+		<actuator name="bust_y_motor">
+			<mechanicalReduction>1</mechanicalReduction>
+		</actuator>
+	</transmission>
+	<link name="chest">
+		<inertial>
+			<origin xyz="2.35256459143538E-06 0.0514948183080913 -0.0105463056982622" rpy="0 0 0"></origin>
+			<mass value="0.0262925523172723"></mass>
+			<inertia ixx="0.000154597294293882" ixy="2.32304239504647E-08" ixz="-2.47140128362103E-08" iyy="0.000750952782458072" iyz="1.53530143139102E-06" izz="0.000688549998744818"></inertia>
+		</inertial>
+		<visual>
+			<origin xyz="0 0 0" rpy="0 0 0"></origin>
+			<geometry>
+				<mesh filename="package://poppy_torso_description/meshes/chest_visual.STL"></mesh>
+			</geometry>
+			<material name="">
+				<color rgba="0.9 0.9 0.9 1.0"></color>
+			</material>
+		</visual>
+		<collision>
+			<origin xyz="0 0 0" rpy="0 0 0"></origin>
+			<geometry>
+				<mesh filename="package://poppy_torso_description/meshes/chest_respondable.STL"></mesh>
+			</geometry>
+		</collision>
+		<mass>0.027528</mass>
+	</link>
+	<joint name="bust_x" type="revolute">
+		<origin xyz="0 0 0" rpy="0 0 0"></origin>
+		<parent link="bust_motors"></parent>
+		<child link="chest"></child>
+		<axis xyz="0 0 1"></axis>
+		<limit lower="-1.0" upper="1.0" effort="10" velocity="3.1415"></limit>
+	</joint>
+	<transmission name="bust_x_trans">
+		<type>transmission_interface/SimpleTransmission</type>
+		<joint name="bust_x">
+			<hardwareInterface>hardware_interface/PositionJointInterface</hardwareInterface>
+		</joint>
+		<actuator name="bust_x_motor">
+			<mechanicalReduction>1</mechanicalReduction>
+		</actuator>
+	</transmission>
+	<link name="neck">
+		<inertial>
+			<origin xyz="-0.00147486363077957 0.00928455262636602 2.89600749219313E-06" rpy="0 0 0"></origin>
+			<mass value="0.000588496516988365"></mass>
+			<inertia ixx="7.25596636570396E-07" ixy="-9.29944216419538E-08" ixz="2.01438227027406E-10" iyy="2.33535976458607E-06" iyz="1.55383710797264E-11" izz="2.57395421284165E-06"></inertia>
+		</inertial>
+		<visual>
+			<origin xyz="0 0 0" rpy="0 0 0"></origin>
+			<geometry>
+				<mesh filename="package://poppy_torso_description/meshes/neck_visual.STL"></mesh>
+			</geometry>
+			<material name="">
+				<color rgba="0.9 0.9 0.9 1.0"></color>
+			</material>
+		</visual>
+		<collision>
+			<origin xyz="0 0 0" rpy="0 0 0"></origin>
+			<geometry>
+				<mesh filename="package://poppy_torso_description/meshes/neck_respondable.STL"></mesh>
+			</geometry>
+		</collision>
+		<mass>0.000588</mass>
+	</link>
+	<joint name="head_z" type="revolute">
+		<origin xyz="0 0.084 0.00499999999999996" rpy="0 0 0"></origin>
+		<parent link="chest"></parent>
+		<child link="neck"></child>
+		<axis xyz="0 1 0"></axis>
+		<limit lower="-1.0" upper="1.0" effort="10" velocity="3.1415"></limit>
+	</joint>
+	<transmission name="head_z_trans">
+		<type>transmission_interface/SimpleTransmission</type>
+		<joint name="head_z">
+			<hardwareInterface>hardware_interface/PositionJointInterface</hardwareInterface>
+		</joint>
+		<actuator name="head_z_motor">
+			<mechanicalReduction>1</mechanicalReduction>
+		</actuator>
+	</transmission>
+	<link name="head">
+		<inertial>
+			<origin xyz="0.000557544173188459 0.0327437693305889 -0.0132545775103434" rpy="0 0 0"></origin>
+			<mass value="0.0188564323997503"></mass>
+			<inertia ixx="0.000353329921483274" ixy="-2.17595216032547E-07" ixz="4.10678991843685E-06" iyy="0.000384587155295662" iyz="-2.16656424152966E-05" izz="0.000396626339401006"></inertia>
+		</inertial>
+		<visual>
+			<origin xyz="0 0 0" rpy="0 0 0"></origin>
+			<geometry>
+				<mesh filename="package://poppy_torso_description/meshes/head_visual.STL"></mesh>
+			</geometry>
+			<material name="">
+				<color rgba="0.9 0.9 0.9 1.0"></color>
+			</material>
+		</visual>
+		<collision>
+			<origin xyz="0 0 0" rpy="0 0 0"></origin>
+			<geometry>
+				<mesh filename="package://poppy_torso_description/meshes/head_respondable.STL"></mesh>
+			</geometry>
+		</collision>
+		<mass>0.02126</mass>
+	</link>
+	<joint name="head_y" type="revolute">
+		<origin xyz="0 0.0199999999999999 0" rpy="-0.349065850398866 0 0"></origin>
+		<parent link="neck"></parent>
+		<child link="head"></child>
+		<axis xyz="-1 0 0"></axis>
+		<limit lower="-0.74" upper="0.2" effort="10" velocity="3.1415"></limit>
+	</joint>
+	<transmission name="head_y_trans">
+		<type>transmission_interface/SimpleTransmission</type>
+		<joint name="head_y">
+			<hardwareInterface>hardware_interface/PositionJointInterface</hardwareInterface>
+		</joint>
+		<actuator name="head_y_motor">
+			<mechanicalReduction>1</mechanicalReduction>
+		</actuator>
+	</transmission>
+	<link name="l_shoulder">
+		<inertial>
+			<origin xyz="0.0105246491971973 0.00179805316216127 -0.00915201992957032" rpy="0 0 0"></origin>
+			<mass value="0.000843598968780806"></mass>
+			<inertia ixx="3.39606863056539E-06" ixy="-4.79545875245114E-08" ixz="2.95435354929514E-08" iyy="3.56726082486902E-06" iyz="1.00382310579659E-08" izz="1.84634806401887E-06"></inertia>
+		</inertial>
+		<visual>
+			<origin xyz="0 0 0" rpy="0 0 0"></origin>
+			<geometry>
+				<mesh filename="package://poppy_torso_description/meshes/l_shoulder_visual.STL"></mesh>
+			</geometry>
+			<material name="">
+				<color rgba="0.9 0.9 0.9 1.0"></color>
+			</material>
+		</visual>
+		<collision>
+			<origin xyz="0 0 0" rpy="0 0 0"></origin>
+			<geometry>
+				<mesh filename="package://poppy_torso_description/meshes/l_shoulder_respondable.STL"></mesh>
+			</geometry>
+		</collision>
+		<mass>0.000838</mass>
+	</link>
+	<joint name="l_shoulder_y" type="revolute">
+		<origin xyz="0.0771000000000001 0.0499999999999999 0.00399999999999997" rpy="-1.5707963267949 0 0"></origin>
+		<parent link="chest"></parent>
+		<child link="l_shoulder"></child>
+		<axis xyz="1 0 0"></axis>
+		<limit lower="-1.8" upper="1.7" effort="10" velocity="3.1415"></limit>
+	</joint>
+	<transmission name="l_shoulder_y_trans">
+		<type>transmission_interface/SimpleTransmission</type>
+		<joint name="l_shoulder_y">
+			<hardwareInterface>hardware_interface/PositionJointInterface</hardwareInterface>
+		</joint>
+		<actuator name="l_shoulder_y_motor">
+			<mechanicalReduction>1</mechanicalReduction>
+		</actuator>
+	</transmission>
+	<link name="l_shoulder_motor">
+		<inertial>
+			<origin xyz="2.25562237481797E-07 0.0125756739553211 0.00859826040204853" rpy="0 0 0"></origin>
+			<mass value="0.00828144098443214"></mass>
+			<inertia ixx="2.76486208811411E-05" ixy="1.32207552337974E-10" ixz="6.6889770978984E-10" iyy="1.64427853426986E-05" iyz="7.23401723852699E-07" izz="2.26416351010788E-05"></inertia>
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