Commit message: fichiers 3d et integration description complète

File: src/poppy_torso_gripper_description/urdf/Poppy_Torso.URDF (robot description, URDF)
Before this commit: robot Poppy_Torso, 14 links, 13 joints
Links:
- added link r_gripper, mass 0.0486511084909604; collision mesh filename=package://poppy_torso_description/meshes/gripper_jaw_respon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; visual mesh filename=package://poppy_torso_description/meshes/gripper_jaw_visual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
- added link world
- link r_forearm: geometry collision mesh filename=package://poppy_torso_description/meshes/forearm_grip_respo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; visual mesh filename=package://poppy_torso_description/meshes/forearm_grip_visua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
Joints:
- added joint fixed: type fixed, parent world, child base
- added joint r_gripper_y: type revolute, parent r_forearm, child r_gripper, origin xyz=0 0.11175 -0.01 rpy=0 0 0, axis -1 0 0, limit lower=-0.0174532925199 upper=2.58308729295 effort=3.1 velocity=7.0
